Commit message: Changed joints in urdfs to NAO convention (right-hand-rule)

File: urdf/complete.urdf (robot description, URDF)
Before this commit: robot complete, 45 links, 44 joints
Links:
- link finger_segment:11: geometry collision mesh filename=package://NICO-models/finger_segment_ipt_50d2a7f4.STL scale=0.001 0.001 0.001; visual mesh filename=package://NICO-models/finger_segment_ipt_50d2a7f4.STL scale=0.001 0.001 0.001
- link finger_segment:12: geometry collision mesh filename=package://NICO-models/finger_segment_ipt_50d2a7f4.STL scale=0.001 0.001 0.001; visual mesh filename=package://NICO-models/finger_segment_ipt_50d2a7f4.STL scale=0.001 0.001 0.001
- link finger_segment:13: geometry collision mesh filename=package://NICO-models/finger_segment_ipt_50d2a7f4.STL scale=0.001 0.001 0.001; visual mesh filename=package://NICO-models/finger_segment_ipt_50d2a7f4.STL scale=0.001 0.001 0.001
- link finger_segment:14: geometry collision mesh filename=package://NICO-models/finger_segment_ipt_50d2a7f4.STL scale=0.001 0.001 0.001; visual mesh filename=package://NICO-models/finger_segment_ipt_50d2a7f4.STL scale=0.001 0.001 0.001
- link finger_segment:15: geometry collision mesh filename=package://NICO-models/finger_segment_ipt_50d2a7f4.STL scale=0.001 0.001 0.001; visual mesh filename=package://NICO-models/finger_segment_ipt_50d2a7f4.STL scale=0.001 0.001 0.001
- link finger_segment:16: geometry collision mesh filename=package://NICO-models/finger_segment_ipt_50d2a7f4.STL scale=0.001 0.001 0.001; visual mesh filename=package://NICO-models/finger_segment_ipt_50d2a7f4.STL scale=0.001 0.001 0.001
- link finger_segment:21: geometry collision mesh filename=package://NICO-models/finger_segment_ipt_50d2a7f4.STL scale=0.001 0.001 0.001; visual mesh filename=package://NICO-models/finger_segment_ipt_50d2a7f4.STL scale=0.001 0.001 0.001
- link finger_segment:22: geometry collision mesh filename=package://NICO-models/finger_segment_ipt_50d2a7f4.STL scale=0.001 0.001 0.001; visual mesh filename=package://NICO-models/finger_segment_ipt_50d2a7f4.STL scale=0.001 0.001 0.001
- link finger_segment:23: geometry collision mesh filename=package://NICO-models/finger_segment_ipt_50d2a7f4.STL scale=0.001 0.001 0.001; visual mesh filename=package://NICO-models/finger_segment_ipt_50d2a7f4.STL scale=0.001 0.001 0.001
- link finger_segment:24: geometry collision mesh filename=package://NICO-models/finger_segment_ipt_50d2a7f4.STL scale=0.001 0.001 0.001; visual mesh filename=package://NICO-models/finger_segment_ipt_50d2a7f4.STL scale=0.001 0.001 0.001
- link finger_segment:25: geometry collision mesh filename=package://NICO-models/finger_segment_ipt_50d2a7f4.STL scale=0.001 0.001 0.001; visual mesh filename=package://NICO-models/finger_segment_ipt_50d2a7f4.STL scale=0.001 0.001 0.001
- link finger_segment:26: geometry collision mesh filename=package://NICO-models/finger_segment_ipt_50d2a7f4.STL scale=0.001 0.001 0.001; visual mesh filename=package://NICO-models/finger_segment_ipt_50d2a7f4.STL scale=0.001 0.001 0.001
- link fingertip:11: geometry collision mesh filename=package://NICO-models/fingertip_ipt_8417b8a9.STL scale=0.001 0.001 0.001; visual mesh filename=package://NICO-models/fingertip_ipt_8417b8a9.STL scale=0.001 0.001 0.001
- link fingertip:12: geometry collision mesh filename=package://NICO-models/fingertip_ipt_8417b8a9.STL scale=0.001 0.001 0.001; visual mesh filename=package://NICO-models/fingertip_ipt_8417b8a9.STL scale=0.001 0.001 0.001
- link fingertip:13: geometry collision mesh filename=package://NICO-models/fingertip_ipt_8417b8a9.STL scale=0.001 0.001 0.001; visual mesh filename=package://NICO-models/fingertip_ipt_8417b8a9.STL scale=0.001 0.001 0.001
- link fingertip:14: geometry collision mesh filename=package://NICO-models/fingertip_ipt_8417b8a9.STL scale=0.001 0.001 0.001; visual mesh filename=package://NICO-models/fingertip_ipt_8417b8a9.STL scale=0.001 0.001 0.001
- link fingertip:15: geometry collision mesh filename=package://NICO-models/fingertip_ipt_8417b8a9.STL scale=0.001 0.001 0.001; visual mesh filename=package://NICO-models/fingertip_ipt_8417b8a9.STL scale=0.001 0.001 0.001
- link fingertip:16: geometry collision mesh filename=package://NICO-models/fingertip_ipt_8417b8a9.STL scale=0.001 0.001 0.001; visual mesh filename=package://NICO-models/fingertip_ipt_8417b8a9.STL scale=0.001 0.001 0.001
- link head:21: geometry collision mesh filename=package://NICO-models/head_iam_b9cf2ea.STL scale=0.001 0.001 0.001; visual mesh filename=package://NICO-models/head_iam_b9cf2ea.STL scale=0.001 0.001 0.001
- link left_ankle:11: geometry collision mesh filename=package://NICO-models/right_ankle_MIR_iam_c5a384f4.STL scale=0.001 0.001 0.001; visual mesh filename=package://NICO-models/right_ankle_MIR_iam_c5a384f4.STL scale=0.001 0.001 0.001
- link left_collarbone:11: geometry collision mesh filename=package://NICO-models/left_upper_arm_iam_49d50008.STL scale=0.001 0.001 0.001; visual mesh filename=package://NICO-models/left_upper_arm_iam_49d50008.STL scale=0.001 0.001 0.001
- link left_foot:11: geometry collision mesh filename=package://NICO-models/left_foot_iam_620666ef.STL scale=0.001 0.001 0.001; visual mesh filename=package://NICO-models/left_foot_iam_620666ef.STL scale=0.001 0.001 0.001
- link left_hip_low:11: geometry collision mesh filename=package://NICO-models/right_hip_up2_MIR_iam_b8a74a0a.STL scale=0.001 0.001 0.001; visual mesh filename=package://NICO-models/right_hip_up2_MIR_iam_b8a74a0a.STL scale=0.001 0.001 0.001
- link left_hip_up:11: geometry collision mesh filename=package://NICO-models/right_hip_up_MIR_iam_386ac7b2.STL scale=0.001 0.001 0.001; visual mesh filename=package://NICO-models/right_hip_up_MIR_iam_386ac7b2.STL scale=0.001 0.001 0.001
- link left_lower_arm:11: geometry collision mesh filename=package://NICO-models/right_wrist_MIR_iam_dcfe6de3.STL scale=0.001 0.001 0.001; visual mesh filename=package://NICO-models/right_wrist_MIR_iam_dcfe6de3.STL scale=0.001 0.001 0.001
- link left_palm:11: geometry collision mesh filename=package://NICO-models/left_palm_iam_b92c61b5.STL scale=0.001 0.001 0.001; visual mesh filename=package://NICO-models/left_palm_iam_b92c61b5.STL scale=0.001 0.001 0.001
- link left_shank:11: geometry collision mesh filename=package://NICO-models/right_shank_MIR_iam_a2a9b5d0.STL scale=0.001 0.001 0.001; visual mesh filename=package://NICO-models/right_shank_MIR_iam_a2a9b5d0.STL scale=0.001 0.001 0.001
- link left_shoulder:11: geometry collision mesh filename=package://NICO-models/left_shoulder_up_iam_1ca4d925.STL scale=0.001 0.001 0.001; visual mesh filename=package://NICO-models/left_shoulder_up_iam_1ca4d925.STL scale=0.001 0.001 0.001
- link left_thigh:11: geometry collision mesh filename=package://NICO-models/Thigh_left_complete_iam_5a6ba909.STL scale=0.001 0.001 0.001; visual mesh filename=package://NICO-models/Thigh_left_complete_iam_5a6ba909.STL scale=0.001 0.001 0.001
- link left_upper_arm:11: geometry collision mesh filename=package://NICO-models/left_lower_arm_iam_5be2a521.STL scale=0.001 0.001 0.001; visual mesh filename=package://NICO-models/left_lower_arm_iam_5be2a521.STL scale=0.001 0.001 0.001
- link left_wrist:11: geometry collision mesh filename=package://NICO-models/left_wrist_iam_c75e4b6f.STL scale=0.001 0.001 0.001; visual mesh filename=package://NICO-models/left_wrist_iam_c75e4b6f.STL scale=0.001 0.001 0.001
- link neck:11: geometry collision mesh filename=package://NICO-models/neck_iam_61141f4f.STL scale=0.001 0.001 0.001; visual mesh filename=package://NICO-models/neck_iam_61141f4f.STL scale=0.001 0.001 0.001
- link right_ankle:11: geometry collision mesh filename=package://NICO-models/right_ankle_iam_f4f7d16a.STL scale=0.001 0.001 0.001; visual mesh filename=package://NICO-models/right_ankle_iam_f4f7d16a.STL scale=0.001 0.001 0.001
- link right_collarbone:11: geometry collision mesh filename=package://NICO-models/right_upper_arm_iam_e3e9c979.STL scale=0.001 0.001 0.001; visual mesh filename=package://NICO-models/right_upper_arm_iam_e3e9c979.STL scale=0.001 0.001 0.001
- link right_foot:11: geometry collision mesh filename=package://NICO-models/right_foot_iam_3ff7356a.STL scale=0.001 0.001 0.001; visual mesh filename=package://NICO-models/right_foot_iam_3ff7356a.STL scale=0.001 0.001 0.001
- link right_hip_low:11: geometry collision mesh filename=package://NICO-models/right_hip_up2_iam_f4f7d16a.STL scale=0.001 0.001 0.001; visual mesh filename=package://NICO-models/right_hip_up2_iam_f4f7d16a.STL scale=0.001 0.001 0.001
- link right_hip_up:11: geometry collision mesh filename=package://NICO-models/right_hip_up_iam_f46f7684.STL scale=0.001 0.001 0.001; visual mesh filename=package://NICO-models/right_hip_up_iam_f46f7684.STL scale=0.001 0.001 0.001
- link right_lower_arm:11: geometry collision mesh filename=package://NICO-models/right_wrist_iam_771ea33e.STL scale=0.001 0.001 0.001; visual mesh filename=package://NICO-models/right_wrist_iam_771ea33e.STL scale=0.001 0.001 0.001
- link right_palm:11: geometry collision mesh filename=package://NICO-models/right_palm_iam_583b22df.STL scale=0.001 0.001 0.001; visual mesh filename=package://NICO-models/right_palm_iam_583b22df.STL scale=0.001 0.001 0.001
- link right_shank:11: geometry collision mesh filename=package://NICO-models/right_shank_iam_7a73fe91.STL scale=0.001 0.001 0.001; visual mesh filename=package://NICO-models/right_shank_iam_7a73fe91.STL scale=0.001 0.001 0.001
- link right_shoulder:11: geometry collision mesh filename=package://NICO-models/right_shoulder_up_iam_34db21c8.STL scale=0.001 0.001 0.001; visual mesh filename=package://NICO-models/right_shoulder_up_iam_34db21c8.STL scale=0.001 0.001 0.001
- link right_thigh:11: geometry collision mesh filename=package://NICO-models/Thigh_right_complete_iam_6502f197.STL scale=0.001 0.001 0.001; visual mesh filename=package://NICO-models/Thigh_right_complete_iam_6502f197.STL scale=0.001 0.001 0.001
- link right_upper_arm:11: geometry collision mesh filename=package://NICO-models/right_lower_arm1_iam_65a34910.STL scale=0.001 0.001 0.001; visual mesh filename=package://NICO-models/right_lower_arm1_iam_65a34910.STL scale=0.001 0.001 0.001
- link right_wrist:11: geometry collision mesh filename=package://NICO-models/right_wrist_iam_81504746.STL scale=0.001 0.001 0.001; visual mesh filename=package://NICO-models/right_wrist_iam_81504746.STL scale=0.001 0.001 0.001
- link torso:11: geometry collision mesh filename=package://NICO-models/torso_iam_fb80b350.STL scale=0.001 0.001 0.001; visual mesh filename=package://NICO-models/torso_iam_fb80b350.STL scale=0.001 0.001 0.001
Joints:
- joint l_ankle_x: axis -1 0 0 -> 1 0 0
- joint l_ankle_y: axis 0 -1 0 -> 0 1 0
- joint l_arm_x: axis -1 0 0 -> 1 0 0; limit lower=-2.05949 upper=1.51844 effort=30 velocity=1 -> lower=-1.51844 upper=2.05949 effort=30 velocity=1
- joint l_elbow_y: axis 0 -1 0 -> 0 1 0
- joint l_hip_x: axis -1 0 0 -> 1 0 0; limit lower=-0.418879 upper=1.22173 effort=30 velocity=1 -> lower=-1.22173 upper=0.418879 effort=30 velocity=1
- joint l_hip_y: axis 0 -1 0 -> 0 1 0; limit lower=-0.698132 upper=1.57 effort=30 velocity=1 -> lower=-1.57 upper=0.698132 effort=30 velocity=1
- joint l_indexfinger_1st_x: axis -0.99794 0.0170003 -0.0618655 -> 0.99794 -0.0170003 0.0618655; limit lower=0 upper=1.309 effort=30 velocity=1 -> lower=-1.309 upper=0 effort=30 velocity=1
- joint l_indexfinger_2nd_x: axis -0.99794 0.0170003 -0.0618655 -> 0.99794 -0.0170003 0.0618655; limit lower=0 upper=1.309 effort=30 velocity=1 -> lower=-1.309 upper=0 effort=30 velocity=1
- joint l_indexfinger_base_x: axis -0.99794 0.0170003 -0.0618655 -> 0.99794 -0.0170003 0.0618655; limit lower=0 upper=1.309 effort=30 velocity=1 -> lower=-1.309 upper=0 effort=30 velocity=1
- joint l_knee_y: axis 0 -1 0 -> 0 1 0; limit lower=-1.29154 upper=1.53589 effort=30 velocity=1 -> lower=-1.53589 upper=1.29154 effort=30 velocity=1
- joint l_palm_x: axis -1 0 0 -> 1 0 0; limit lower=0 upper=0.872665 effort=30 velocity=1 -> lower=-0.872665 upper=0 effort=30 velocity=1
- joint l_ringfinger_1st_x: axis -0.998051 -0.00234199 0.0623629 -> 0.998051 0.00234199 -0.0623629; limit lower=0 upper=1.309 effort=30 velocity=1 -> lower=-1.309 upper=0 effort=30 velocity=1
- joint l_ringfinger_2nd_x: axis -0.998051 -0.00234199 0.0623629 -> 0.998051 0.00234199 -0.0623629; limit lower=0 upper=1.309 effort=30 velocity=1 -> lower=-1.309 upper=0 effort=30 velocity=1
- joint l_ringfinger_base_x: axis -0.998051 -0.00234199 0.0623629 -> 0.998051 0.00234199 -0.0623629; limit lower=0 upper=1.309 effort=30 velocity=1 -> lower=-1.309 upper=0 effort=30 velocity=1
- joint l_shoulder_y: axis 0 -1 0 -> 0 1 0; limit lower=-0.523599 upper=2.79253 effort=30 velocity=1 -> lower=-2.79253 upper=0.523599 effort=30 velocity=1
- joint l_shoulder_z: axis 0 0 -1 -> 0 0 1; limit lower=-1.22173 upper=0.872665 effort=30 velocity=1 -> lower=-0.872665 upper=1.22173 effort=30 velocity=1
- joint l_thumb_1st_x: axis -1 0 0 -> 1 0 0; limit lower=-0.872665 upper=0.610865 effort=30 velocity=1 -> lower=-1.309 upper=0 effort=30 velocity=1
- joint l_thumb_2nd_x: axis -1 0 0 -> 1 0 0; limit lower=-0.872665 upper=0.610865 effort=30 velocity=1 -> lower=-1.309 upper=0 effort=30 velocity=1
- joint l_thumb_base_x: axis -1 0 0 -> 1 0 0; limit lower=-0.872665 upper=0.610865 effort=30 velocity=1 -> lower=-1.309 upper=0 effort=30 velocity=1
- joint l_wrist_z: axis 0 0 -1 -> 0 0 1
- joint r_ankle_y: axis 0 -1 0 -> 0 1 0
- joint r_hip_y: axis 0 -1 0 -> 0 1 0; limit lower=-0.5585 upper=1.570796 effort=30 velocity=1 -> lower=-1.570796 upper=0.5585 effort=30 velocity=1
- joint r_indexfinger_1st_x: axis -0.998022 -0.00962907 -0.0621208 -> 0.998022 0.00962907 0.0621208; limit lower=0 upper=1.309 effort=30 velocity=1 -> lower=-1.309 upper=0 effort=30 velocity=1
- joint r_indexfinger_2nd_x: axis -0.998022 -0.00962907 -0.0621208 -> 0.998022 0.00962907 0.0621208; limit lower=0 upper=1.309 effort=30 velocity=1 -> lower=-1.309 upper=0 effort=30 velocity=1
- joint r_indexfinger_base_x: axis -0.998022 -0.00962907 -0.0621208 -> 0.998022 0.00962907 0.0621208; limit lower=0 upper=1.309 effort=30 velocity=1 -> lower=-1.309 upper=0 effort=30 velocity=1
- joint r_knee_y: axis 0 -1 0 -> 0 1 0; limit lower=-1.29154 upper=1.53589 effort=30 velocity=1 -> lower=-1.53589 upper=1.29154 effort=30 velocity=1
- joint r_ringfinger_1st_x: axis -0.998022 0.00962907 0.0621208 -> 0.998022 -0.00962907 -0.0621208; limit lower=0 upper=1.309 effort=30 velocity=1 -> lower=-1.309 upper=0 effort=30 velocity=1
- joint r_ringfinger_2nd_x: axis -0.998022 0.00962907 0.0621208 -> 0.998022 -0.00962907 -0.0621208; limit lower=0 upper=1.309 effort=30 velocity=1 -> lower=-1.309 upper=0 effort=30 velocity=1
- joint r_ringfinger_base_x: axis -0.998022 0.00962907 0.0621208 -> 0.998022 -0.00962907 -0.0621208; limit lower=0 upper=1.309 effort=30 velocity=1 -> lower=-1.309 upper=0 effort=30 velocity=1
- joint r_shoulder_y: axis 0 -1 0 -> 0 1 0; limit lower=-0.523599 upper=2.79253 effort=30 velocity=1 -> lower=-2.79253 upper=0.523599 effort=30 velocity=1
- joint r_thumb_1st_x: axis -1 0 0 -> 1 0 0; limit lower=0 upper=1.309 effort=30 velocity=1 -> lower=-1.309 upper=0 effort=30 velocity=1
- joint r_thumb_2nd_x: axis -1 0 0 -> 1 0 0; limit lower=0 upper=1.309 effort=30 velocity=1 -> lower=-1.309 upper=0 effort=30 velocity=1
- joint r_thumb_base_x: axis -1 0 0 -> 1 0 0; limit lower=0 upper=1.309 effort=30 velocity=1 -> lower=-1.309 upper=0 effort=30 velocity=1

File: urdf/seed_hand.urdf (robot description, URDF)
Before this commit: robot seed_hand, 11 links, 10 joints
Links:
- link finger_segment:11: geometry collision mesh filename=package://NICO-models/finger_segment_ipt_50d2a7f4.STL scale=0.001 0.001 0.001; visual mesh filename=package://NICO-models/finger_segment_ipt_50d2a7f4.STL scale=0.001 0.001 0.001
- link finger_segment:12: geometry collision mesh filename=package://NICO-models/finger_segment_ipt_50d2a7f4.STL scale=0.001 0.001 0.001; visual mesh filename=package://NICO-models/finger_segment_ipt_50d2a7f4.STL scale=0.001 0.001 0.001
- link finger_segment:13: geometry collision mesh filename=package://NICO-models/finger_segment_ipt_50d2a7f4.STL scale=0.001 0.001 0.001; visual mesh filename=package://NICO-models/finger_segment_ipt_50d2a7f4.STL scale=0.001 0.001 0.001
- link finger_segment:21: geometry collision mesh filename=package://NICO-models/finger_segment_ipt_50d2a7f4.STL scale=0.001 0.001 0.001; visual mesh filename=package://NICO-models/finger_segment_ipt_50d2a7f4.STL scale=0.001 0.001 0.001
- link finger_segment:22: geometry collision mesh filename=package://NICO-models/finger_segment_ipt_50d2a7f4.STL scale=0.001 0.001 0.001; visual mesh filename=package://NICO-models/finger_segment_ipt_50d2a7f4.STL scale=0.001 0.001 0.001
- link finger_segment:23: geometry collision mesh filename=package://NICO-models/finger_segment_ipt_50d2a7f4.STL scale=0.001 0.001 0.001; visual mesh filename=package://NICO-models/finger_segment_ipt_50d2a7f4.STL scale=0.001 0.001 0.001
- link fingertip:11: geometry collision mesh filename=package://NICO-models/fingertip_ipt_8417b8a9.STL scale=0.001 0.001 0.001; visual mesh filename=package://NICO-models/fingertip_ipt_8417b8a9.STL scale=0.001 0.001 0.001
- link fingertip:12: geometry collision mesh filename=package://NICO-models/fingertip_ipt_8417b8a9.STL scale=0.001 0.001 0.001; visual mesh filename=package://NICO-models/fingertip_ipt_8417b8a9.STL scale=0.001 0.001 0.001
- link fingertip:13: geometry collision mesh filename=package://NICO-models/fingertip_ipt_8417b8a9.STL scale=0.001 0.001 0.001; visual mesh filename=package://NICO-models/fingertip_ipt_8417b8a9.STL scale=0.001 0.001 0.001
- link right_palm:11: geometry collision mesh filename=package://NICO-models/right_palm_iam_583b22df.STL scale=0.001 0.001 0.001; visual mesh filename=package://NICO-models/right_palm_iam_583b22df.STL scale=0.001 0.001 0.001
- link right_wrist:11: geometry collision mesh filename=package://NICO-models/right_wrist_iam_81504746.STL scale=0.001 0.001 0.001; visual mesh filename=package://NICO-models/right_wrist_iam_81504746.STL scale=0.001 0.001 0.001
Joints:
- joint r_indexfinger_1st_x: axis -0.998022 -0.00962907 -0.0621208 -> 0.998022 0.00962907 0.0621208; limit lower=0 upper=1.309 effort=30 velocity=1 -> lower=-1.309 upper=0 effort=30 velocity=1
- joint r_indexfinger_2nd_x: axis -0.998022 -0.00962907 -0.0621208 -> 0.998022 0.00962907 0.0621208; limit lower=0 upper=1.309 effort=30 velocity=1 -> lower=-1.309 upper=0 effort=30 velocity=1
- joint r_indexfinger_base_x: axis -0.998022 -0.00962907 -0.0621208 -> 0.998022 0.00962907 0.0621208; limit lower=0 upper=1.309 effort=30 velocity=1 -> lower=-1.309 upper=0 effort=30 velocity=1
- joint r_ringfinger_1st_x: axis -0.998022 0.00962907 0.0621208 -> 0.998022 -0.00962907 -0.0621208; limit lower=0 upper=1.309 effort=30 velocity=1 -> lower=-1.309 upper=0 effort=30 velocity=1
- joint r_ringfinger_2nd_x: axis -0.998022 0.00962907 0.0621208 -> 0.998022 -0.00962907 -0.0621208; limit lower=0 upper=1.309 effort=30 velocity=1 -> lower=-1.309 upper=0 effort=30 velocity=1
- joint r_ringfinger_base_x: axis -0.998022 0.00962907 0.0621208 -> 0.998022 -0.00962907 -0.0621208; limit lower=0 upper=1.309 effort=30 velocity=1 -> lower=-1.309 upper=0 effort=30 velocity=1
- joint r_thumb_1st_x: axis -1 0 0 -> 1 0 0; limit lower=0 upper=1.309 effort=30 velocity=1 -> lower=-1.309 upper=0 effort=30 velocity=1
- joint r_thumb_2nd_x: axis -1 0 0 -> 1 0 0; limit lower=0 upper=1.309 effort=30 velocity=1 -> lower=-1.309 upper=0 effort=30 velocity=1
- joint r_thumb_base_x: axis -1 0 0 -> 1 0 0; limit lower=0 upper=1.309 effort=30 velocity=1 -> lower=-1.309 upper=0 effort=30 velocity=1

Commit message: fixed finger distance of left hand to match the right

File: urdf/complete.urdf (robot description, URDF)
Before this commit: robot complete, 45 links, 44 joints
Joints:
- joint l_indexfinger_1st_x: axis 0.99794 -0.0170003 0.0618655 -> 0.99794 -0.0170003 -0.0618655
- joint l_indexfinger_2nd_x: axis 0.99794 -0.0170003 0.0618655 -> 0.99794 -0.0170003 -0.0618655
- joint l_indexfinger_base_x: axis 0.99794 -0.0170003 0.0618655 -> 0.99794 -0.0170003 -0.0618655
- joint l_ringfinger_1st_x: axis 0.998051 0.00234199 -0.0623629 -> 0.998051 0.00234199 0.0623629
- joint l_ringfinger_2nd_x: axis 0.998051 0.00234199 -0.0623629 -> 0.998051 0.00234199 0.0623629
- joint l_ringfinger_base_x: axis 0.998051 0.00234199 -0.0623629 -> 0.998051 0.00234199 0.0623629

Commit message: URDF synchronized

File: urdf/complete.urdf (robot description, URDF)
Before this commit: robot complete, 45 links, 44 joints
Joints:
- joint head_y: limit lower=-0.785398 upper=0.314159 effort=30 velocity=1 -> lower=-1.553 upper=1.379 effort=30 velocity=1
- joint head_z: limit lower=-2.18166 upper=2.18166 effort=30 velocity=1 -> lower=-3.124 upper=3.142 effort=30 velocity=1
- joint l_arm_x: limit lower=-1.51844 upper=2.05949 effort=30 velocity=1 -> lower=-1.8675 upper=3.002 effort=30 velocity=1
- joint l_elbow_y: axis 0 1 0 -> 0 -1 0; limit lower=-1.5708 upper=1.5708 effort=30 velocity=1 -> lower=-1.745 upper=1.745 effort=30 velocity=1
- joint l_hip_z: axis 0 0 -1 -> 0 0 1
- joint l_shoulder_y: limit lower=-2.79253 upper=0.523599 effort=30 velocity=1 -> lower=-3.124 upper=3.142 effort=30 velocity=1
- joint l_shoulder_z: limit lower=-0.872665 upper=1.22173 effort=30 velocity=1 -> lower=-2.182 upper=1.745 effort=30 velocity=1
- joint l_wrist_z: axis 0 0 1 -> 0 0 -1; limit lower=-1.5708 upper=1.5708 effort=30 velocity=1 -> lower=-1.571 upper=1.571 effort=30 velocity=1
- joint r_arm_x: limit lower=-2.05949 upper=1.51844 effort=30 velocity=1 -> lower=-1.885 upper=0.751 effort=30 velocity=1
- joint r_elbow_y: axis 0 -1 0 -> 0 1 0; limit lower=-1.5708 upper=1.5708 effort=30 velocity=1 -> lower=-1.745 upper=1.745 effort=30 velocity=1
- joint r_shoulder_y: axis 0 1 0 -> 0 -1 0; limit lower=-2.79253 upper=0.523599 effort=30 velocity=1 -> lower=-3.142 upper=3.124 effort=30 velocity=1
- joint r_shoulder_z: limit lower=-1.22173 upper=0.872665 effort=30 velocity=1 -> lower=-1.745 upper=2.182 effort=30 velocity=1
- joint r_wrist_z: axis 0 0 -1 -> 0 0 1; limit lower=-1.5708 upper=1.5708 effort=30 velocity=1 -> lower=-1.571 upper=1.571 effort=30 velocity=1

Commit message: limits for r_arm_x corrected in urdf

File: urdf/complete.urdf (robot description, URDF)
Before this commit: robot complete, 45 links, 44 joints
Joints:
- joint r_arm_x: limit lower=-1.885 upper=0.751 effort=30 velocity=1 -> lower=-3.002 upper=1.8675 effort=30 velocity=1
