Commit message: renamed finger joints

File: urdf/complete.urdf (robot description, URDF)
Before this commit: robot complete, 45 links, 44 joints
Joints:
- removed joint l_indexfinger_base_x
- removed joint l_ringfinger_base_x
- removed joint l_thumb_base_x
- removed joint r_indexfinger_base_x
- removed joint r_ringfinger_base_x
- removed joint r_thumb_base_x
- added joint l_indexfingers_x: type revolute, parent left_palm:11, child finger_segment:25, origin xyz=-0.001439 0.006226 0.040004 rpy=2.492946 0.062904 0, axis 0.99794 -0.0170003 -0.0618655, limit lower=-1.309 upper=0 effort=30 velocity=1
- added joint l_ringfingers_x: type revolute, parent left_palm:11, child finger_segment:26, origin xyz=-0.036179 0.006226 0.04057 rpy=2.499505 -0.062904 0, axis 0.998051 0.00234199 0.0623629, limit lower=-1.309 upper=0 effort=30 velocity=1
- added joint l_thumb_x: type revolute, parent left_palm:11, child finger_segment:24, origin xyz=-0.028 0.0199 0.00842 rpy=-1.130534 0 -3.141593, axis 1 0 0, limit lower=-1.309 upper=0 effort=30 velocity=1
- added joint r_indexfingers_x: type revolute, parent right_palm:11, child finger_segment:23, origin xyz=-0.001139 0.006226 -0.040004 rpy=-0.578103 0.062904 -3.141593, axis 0.998022 0.00962907 0.0621208, limit lower=-1.309 upper=0 effort=30 velocity=1
- added joint r_ringfingers_x: type revolute, parent right_palm:11, child finger_segment:22, origin xyz=-0.035879 0.006226 -0.040569 rpy=-0.569851 -0.062904 -3.141593, axis 0.998022 -0.00962907 -0.0621208, limit lower=-1.309 upper=0 effort=30 velocity=1
- added joint r_thumb_x: type revolute, parent right_palm:11, child finger_segment:21, origin xyz=-0.0275 0.0199 -0.00842 rpy=1.915504 0 0, axis 1 0 0, limit lower=-1.309 upper=0 effort=30 velocity=1

Commit message: renamed palm_x --> wrist_x

File: urdf/complete.urdf (robot description, URDF)
Before this commit: robot complete, 45 links, 44 joints
Joints:
- removed joint l_palm_x
- removed joint r_palm_x
- added joint l_wrist_x: type revolute, parent left_wrist:11, child left_palm:11, origin xyz=0.023416 0.006052 0.070837 rpy=0.460941 0 0, axis 1 0 0, limit lower=-0.872665 upper=0 effort=30 velocity=1
- added joint r_wrist_x: type revolute, parent right_wrist:11, child right_palm:11, origin xyz=0.023416 0.006052 -0.070337 rpy=-0.433097 0 0, axis 1 0 0, limit lower=0 upper=0.872665 effort=30 velocity=1

Commit message: urdf folder cleanup

File: urdf/complete.urdf (robot description, URDF)
Before this commit: robot complete, 45 links, 44 joints
Links:
- link finger_segment:11: geometry collision mesh filename=package://NICO-models/meshes/finger_segment_ipt_50d2a7f4.STL scale=0.001 0.001 0.001; visual mesh filename=package://NICO-models/meshes/finger_segment_ipt_50d2a7f4.STL scale=0.001 0.001 0.001
- link finger_segment:12: geometry collision mesh filename=package://NICO-models/meshes/finger_segment_ipt_50d2a7f4.STL scale=0.001 0.001 0.001; visual mesh filename=package://NICO-models/meshes/finger_segment_ipt_50d2a7f4.STL scale=0.001 0.001 0.001
- link finger_segment:13: geometry collision mesh filename=package://NICO-models/meshes/finger_segment_ipt_50d2a7f4.STL scale=0.001 0.001 0.001; visual mesh filename=package://NICO-models/meshes/finger_segment_ipt_50d2a7f4.STL scale=0.001 0.001 0.001
- link finger_segment:14: geometry collision mesh filename=package://NICO-models/meshes/finger_segment_ipt_50d2a7f4.STL scale=0.001 0.001 0.001; visual mesh filename=package://NICO-models/meshes/finger_segment_ipt_50d2a7f4.STL scale=0.001 0.001 0.001
- link finger_segment:15: geometry collision mesh filename=package://NICO-models/meshes/finger_segment_ipt_50d2a7f4.STL scale=0.001 0.001 0.001; visual mesh filename=package://NICO-models/meshes/finger_segment_ipt_50d2a7f4.STL scale=0.001 0.001 0.001
- link finger_segment:16: geometry collision mesh filename=package://NICO-models/meshes/finger_segment_ipt_50d2a7f4.STL scale=0.001 0.001 0.001; visual mesh filename=package://NICO-models/meshes/finger_segment_ipt_50d2a7f4.STL scale=0.001 0.001 0.001
- link finger_segment:21: geometry collision mesh filename=package://NICO-models/meshes/finger_segment_ipt_50d2a7f4.STL scale=0.001 0.001 0.001; visual mesh filename=package://NICO-models/meshes/finger_segment_ipt_50d2a7f4.STL scale=0.001 0.001 0.001
- link finger_segment:22: geometry collision mesh filename=package://NICO-models/meshes/finger_segment_ipt_50d2a7f4.STL scale=0.001 0.001 0.001; visual mesh filename=package://NICO-models/meshes/finger_segment_ipt_50d2a7f4.STL scale=0.001 0.001 0.001
- link finger_segment:23: geometry collision mesh filename=package://NICO-models/meshes/finger_segment_ipt_50d2a7f4.STL scale=0.001 0.001 0.001; visual mesh filename=package://NICO-models/meshes/finger_segment_ipt_50d2a7f4.STL scale=0.001 0.001 0.001
- link finger_segment:24: geometry collision mesh filename=package://NICO-models/meshes/finger_segment_ipt_50d2a7f4.STL scale=0.001 0.001 0.001; visual mesh filename=package://NICO-models/meshes/finger_segment_ipt_50d2a7f4.STL scale=0.001 0.001 0.001
- link finger_segment:25: geometry collision mesh filename=package://NICO-models/meshes/finger_segment_ipt_50d2a7f4.STL scale=0.001 0.001 0.001; visual mesh filename=package://NICO-models/meshes/finger_segment_ipt_50d2a7f4.STL scale=0.001 0.001 0.001
- link finger_segment:26: geometry collision mesh filename=package://NICO-models/meshes/finger_segment_ipt_50d2a7f4.STL scale=0.001 0.001 0.001; visual mesh filename=package://NICO-models/meshes/finger_segment_ipt_50d2a7f4.STL scale=0.001 0.001 0.001
- link fingertip:11: geometry collision mesh filename=package://NICO-models/meshes/fingertip_ipt_8417b8a9.STL scale=0.001 0.001 0.001; visual mesh filename=package://NICO-models/meshes/fingertip_ipt_8417b8a9.STL scale=0.001 0.001 0.001
- link fingertip:12: geometry collision mesh filename=package://NICO-models/meshes/fingertip_ipt_8417b8a9.STL scale=0.001 0.001 0.001; visual mesh filename=package://NICO-models/meshes/fingertip_ipt_8417b8a9.STL scale=0.001 0.001 0.001
- link fingertip:13: geometry collision mesh filename=package://NICO-models/meshes/fingertip_ipt_8417b8a9.STL scale=0.001 0.001 0.001; visual mesh filename=package://NICO-models/meshes/fingertip_ipt_8417b8a9.STL scale=0.001 0.001 0.001
- link fingertip:14: geometry collision mesh filename=package://NICO-models/meshes/fingertip_ipt_8417b8a9.STL scale=0.001 0.001 0.001; visual mesh filename=package://NICO-models/meshes/fingertip_ipt_8417b8a9.STL scale=0.001 0.001 0.001
- link fingertip:15: geometry collision mesh filename=package://NICO-models/meshes/fingertip_ipt_8417b8a9.STL scale=0.001 0.001 0.001; visual mesh filename=package://NICO-models/meshes/fingertip_ipt_8417b8a9.STL scale=0.001 0.001 0.001
- link fingertip:16: geometry collision mesh filename=package://NICO-models/meshes/fingertip_ipt_8417b8a9.STL scale=0.001 0.001 0.001; visual mesh filename=package://NICO-models/meshes/fingertip_ipt_8417b8a9.STL scale=0.001 0.001 0.001
- link head:21: geometry collision mesh filename=package://NICO-models/meshes/head_iam_b9cf2ea.STL scale=0.001 0.001 0.001; visual mesh filename=package://NICO-models/meshes/head_iam_b9cf2ea.STL scale=0.001 0.001 0.001
- link left_ankle:11: geometry collision mesh filename=package://NICO-models/meshes/right_ankle_MIR_iam_c5a384f4.S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 scale=0.001 0.001 0.001; visual mesh filename=package://NICO-models/meshes/right_ankle_MIR_iam_c5a384f4.S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 scale=0.001 0.001 0.001
- link left_collarbone:11: geometry collision mesh filename=package://NICO-models/meshes/left_upper_arm_iam_49d50008.STL scale=0.001 0.001 0.001; visual mesh filename=package://NICO-models/meshes/left_upper_arm_iam_49d50008.STL scale=0.001 0.001 0.001
- link left_foot:11: geometry collision mesh filename=package://NICO-models/meshes/left_foot_iam_620666ef.STL scale=0.001 0.001 0.001; visual mesh filename=package://NICO-models/meshes/left_foot_iam_620666ef.STL scale=0.001 0.001 0.001
- link left_hip_low:11: geometry collision mesh filename=package://NICO-models/meshes/right_hip_up2_MIR_iam_b8a74a0a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 scale=0.001 0.001 0.001; visual mesh filename=package://NICO-models/meshes/right_hip_up2_MIR_iam_b8a74a0a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 scale=0.001 0.001 0.001
- link left_hip_up:11: geometry collision mesh filename=package://NICO-models/meshes/right_hip_up_MIR_iam_386ac7b2.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 scale=0.001 0.001 0.001; visual mesh filename=package://NICO-models/meshes/right_hip_up_MIR_iam_386ac7b2.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 scale=0.001 0.001 0.001
- link left_lower_arm:11: geometry collision mesh filename=package://NICO-models/meshes/right_wrist_MIR_iam_dcfe6de3.S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 scale=0.001 0.001 0.001; visual mesh filename=package://NICO-models/meshes/right_wrist_MIR_iam_dcfe6de3.S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 scale=0.001 0.001 0.001
- link left_palm:11: geometry collision mesh filename=package://NICO-models/meshes/left_palm_iam_b92c61b5.STL scale=0.001 0.001 0.001; visual mesh filename=package://NICO-models/meshes/left_palm_iam_b92c61b5.STL scale=0.001 0.001 0.001
- link left_shank:11: geometry collision mesh filename=package://NICO-models/meshes/right_shank_MIR_iam_a2a9b5d0.S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 scale=0.001 0.001 0.001; visual mesh filename=package://NICO-models/meshes/right_shank_MIR_iam_a2a9b5d0.S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 scale=0.001 0.001 0.001
- link left_shoulder:11: geometry collision mesh filename=package://NICO-models/meshes/left_shoulder_up_iam_1ca4d925.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 scale=0.001 0.001 0.001; visual mesh filename=package://NICO-models/meshes/left_shoulder_up_iam_1ca4d925.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 scale=0.001 0.001 0.001
- link left_thigh:11: geometry collision mesh filename=package://NICO-models/meshes/Thigh_left_complete_iam_5a6ba9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 scale=0.001 0.001 0.001; visual mesh filename=package://NICO-models/meshes/Thigh_left_complete_iam_5a6ba9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 scale=0.001 0.001 0.001
- link left_upper_arm:11: geometry collision mesh filename=package://NICO-models/meshes/left_lower_arm_iam_5be2a521.STL scale=0.001 0.001 0.001; visual mesh filename=package://NICO-models/meshes/left_lower_arm_iam_5be2a521.STL scale=0.001 0.001 0.001
- link left_wrist:11: geometry collision mesh filename=package://NICO-models/meshes/left_wrist_iam_c75e4b6f.STL scale=0.001 0.001 0.001; visual mesh filename=package://NICO-models/meshes/left_wrist_iam_c75e4b6f.STL scale=0.001 0.001 0.001
- link neck:11: geometry collision mesh filename=package://NICO-models/meshes/neck_iam_61141f4f.STL scale=0.001 0.001 0.001; visual mesh filename=package://NICO-models/meshes/neck_iam_61141f4f.STL scale=0.001 0.001 0.001
- link right_ankle:11: geometry collision mesh filename=package://NICO-models/meshes/right_ankle_iam_f4f7d16a.STL scale=0.001 0.001 0.001; visual mesh filename=package://NICO-models/meshes/right_ankle_iam_f4f7d16a.STL scale=0.001 0.001 0.001
- link right_collarbone:11: geometry collision mesh filename=package://NICO-models/meshes/right_upper_arm_iam_e3e9c979.S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 scale=0.001 0.001 0.001; visual mesh filename=package://NICO-models/meshes/right_upper_arm_iam_e3e9c979.S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 scale=0.001 0.001 0.001
- link right_foot:11: geometry collision mesh filename=package://NICO-models/meshes/right_foot_iam_3ff7356a.STL scale=0.001 0.001 0.001; visual mesh filename=package://NICO-models/meshes/right_foot_iam_3ff7356a.STL scale=0.001 0.001 0.001
- link right_hip_low:11: geometry collision mesh filename=package://NICO-models/meshes/right_hip_up2_iam_f4f7d16a.STL scale=0.001 0.001 0.001; visual mesh filename=package://NICO-models/meshes/right_hip_up2_iam_f4f7d16a.STL scale=0.001 0.001 0.001
- link right_hip_up:11: geometry collision mesh filename=package://NICO-models/meshes/right_hip_up_iam_f46f7684.STL scale=0.001 0.001 0.001; visual mesh filename=package://NICO-models/meshes/right_hip_up_iam_f46f7684.STL scale=0.001 0.001 0.001
- link right_lower_arm:11: geometry collision mesh filename=package://NICO-models/meshes/right_wrist_iam_771ea33e.STL scale=0.001 0.001 0.001; visual mesh filename=package://NICO-models/meshes/right_wrist_iam_771ea33e.STL scale=0.001 0.001 0.001
- link right_palm:11: geometry collision mesh filename=package://NICO-models/meshes/right_palm_iam_583b22df.STL scale=0.001 0.001 0.001; visual mesh filename=package://NICO-models/meshes/right_palm_iam_583b22df.STL scale=0.001 0.001 0.001
- link right_shank:11: geometry collision mesh filename=package://NICO-models/meshes/right_shank_iam_7a73fe91.STL scale=0.001 0.001 0.001; visual mesh filename=package://NICO-models/meshes/right_shank_iam_7a73fe91.STL scale=0.001 0.001 0.001
- link right_shoulder:11: geometry collision mesh filename=package://NICO-models/meshes/right_shoulder_up_iam_34db21c8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 scale=0.001 0.001 0.001; visual mesh filename=package://NICO-models/meshes/right_shoulder_up_iam_34db21c8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 scale=0.001 0.001 0.001
- link right_thigh:11: geometry collision mesh filename=package://NICO-models/meshes/Thigh_right_complete_iam_6502f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 scale=0.001 0.001 0.001; visual mesh filename=package://NICO-models/meshes/Thigh_right_complete_iam_6502f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 scale=0.001 0.001 0.001
- link right_upper_arm:11: geometry collision mesh filename=package://NICO-models/meshes/right_lower_arm1_iam_65a34910.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 scale=0.001 0.001 0.001; visual mesh filename=package://NICO-models/meshes/right_lower_arm1_iam_65a34910.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 scale=0.001 0.001 0.001
- link right_wrist:11: geometry collision mesh filename=package://NICO-models/meshes/right_wrist_iam_81504746.STL scale=0.001 0.001 0.001; visual mesh filename=package://NICO-models/meshes/right_wrist_iam_81504746.STL scale=0.001 0.001 0.001
- link torso:11: geometry collision mesh filename=package://NICO-models/meshes/torso_iam_fb80b350.STL scale=0.001 0.001 0.001; visual mesh filename=package://NICO-models/meshes/torso_iam_fb80b350.STL scale=0.001 0.001 0.001
