Commit message: Updates to Motion, Moveit and setup
-Minor fixes to setup, added missing requirements
-fixed outdated moveit module
-updated json files, added seperate json for vrep
-added angle remapping for hand motors to motion to reflect real angles
-added support for Palm IR sensors to motion

File: api/src/nicomoveit/moveiturdf/urdf/complete.urdf (robot description, URDF)
Before this commit: robot complete, 46 links, 45 joints
Links:
- link head:21: geometry collision mesh filename=package://nicoros/../../../urdf/meshes/head_iam_b9cf2ea.STL scale=0.001 0.001 0.001; visual mesh filename=package://nicoros/../../../urdf/meshes/head_iam_b9cf2ea.STL scale=0.001 0.001 0.001
- link left_ankle:11: geometry collision mesh filename=package://nicoros/../../../urdf/meshes/right_ankle_MIR_iam_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 scale=0.001 0.001 0.001; visual mesh filename=package://nicoros/../../../urdf/meshes/right_ankle_MIR_iam_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 scale=0.001 0.001 0.001
- link left_foot:11: geometry collision mesh filename=package://nicoros/../../../urdf/meshes/left_foot_iam_620666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 scale=0.001 0.001 0.001; visual mesh filename=package://nicoros/../../../urdf/meshes/left_foot_iam_620666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 scale=0.001 0.001 0.001
- link left_hip_low:11: geometry collision mesh filename=package://nicoros/../../../urdf/meshes/right_hip_up2_MIR_ia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 scale=0.001 0.001 0.001; visual mesh filename=package://nicoros/../../../urdf/meshes/right_hip_up2_MIR_ia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 scale=0.001 0.001 0.001
- link left_hip_up:11: geometry collision mesh filename=package://nicoros/../../../urdf/meshes/right_hip_up_MIR_iam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 scale=0.001 0.001 0.001; visual mesh filename=package://nicoros/../../../urdf/meshes/right_hip_up_MIR_iam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 scale=0.001 0.001 0.001
- link left_lower_arm:11: geometry collision mesh filename=package://nicoros/../../../urdf/meshes/right_wrist_MIR_iam_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 scale=0.001 0.001 0.001; visual mesh filename=package://nicoros/../../../urdf/meshes/right_wrist_MIR_iam_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 scale=0.001 0.001 0.001
- link left_palm:11: geometry collision mesh filename=package://nicoros/../../../urdf/meshes/left_palm_iam_b92c61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 scale=0.001 0.001 0.001; visual mesh filename=package://nicoros/../../../urdf/meshes/left_palm_iam_b92c61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 scale=0.001 0.001 0.001
- link left_shank:11: geometry collision mesh filename=package://nicoros/../../../urdf/meshes/right_shank_MIR_iam_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 scale=0.001 0.001 0.001; visual mesh filename=package://nicoros/../../../urdf/meshes/right_shank_MIR_iam_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 scale=0.001 0.001 0.001
- link left_shoulder:11: geometry collision mesh filename=package://nicoros/../../../urdf/meshes/left_shoulder_up_iam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 scale=0.001 0.001 0.001; visual mesh filename=package://nicoros/../../../urdf/meshes/left_shoulder_up_iam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 scale=0.001 0.001 0.001
- link left_thigh:11: geometry collision mesh filename=package://nicoros/../../../urdf/meshes/Thigh_left_complete_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 scale=0.001 0.001 0.001; visual mesh filename=package://nicoros/../../../urdf/meshes/Thigh_left_complete_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 scale=0.001 0.001 0.001
- link left_upper_arm:11: geometry collision mesh filename=package://nicoros/../../../urdf/meshes/left_lower_arm_iam_5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 scale=0.001 0.001 0.001; visual mesh filename=package://nicoros/../../../urdf/meshes/left_lower_arm_iam_5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 scale=0.001 0.001 0.001
- link neck:11: geometry collision mesh filename=package://nicoros/../../../urdf/meshes/neck_iam_61141f4f.STL scale=0.001 0.001 0.001; visual mesh filename=package://nicoros/../../../urdf/meshes/neck_iam_61141f4f.STL scale=0.001 0.001 0.001
- link right_ankle:11: geometry collision mesh filename=package://nicoros/../../../urdf/meshes/right_ankle_iam_f4f7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 scale=0.001 0.001 0.001; visual mesh filename=package://nicoros/../../../urdf/meshes/right_ankle_iam_f4f7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 scale=0.001 0.001 0.001
- link right_foot:11: geometry collision mesh filename=package://nicoros/../../../urdf/meshes/right_foot_iam_3ff73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 scale=0.001 0.001 0.001; visual mesh filename=package://nicoros/../../../urdf/meshes/right_foot_iam_3ff73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 scale=0.001 0.001 0.001
- link right_hip_low:11: geometry collision mesh filename=package://nicoros/../../../urdf/meshes/right_hip_up2_iam_f4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 scale=0.001 0.001 0.001; visual mesh filename=package://nicoros/../../../urdf/meshes/right_hip_up2_iam_f4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 scale=0.001 0.001 0.001
- link right_hip_up:11: geometry collision mesh filename=package://nicoros/../../../urdf/meshes/right_hip_up_iam_f46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 scale=0.001 0.001 0.001; visual mesh filename=package://nicoros/../../../urdf/meshes/right_hip_up_iam_f46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 scale=0.001 0.001 0.001
- link right_lower_arm:11: geometry collision mesh filename=package://nicoros/../../../urdf/meshes/right_wrist_iam_771e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 scale=0.001 0.001 0.001; visual mesh filename=package://nicoros/../../../urdf/meshes/right_wrist_iam_771e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 scale=0.001 0.001 0.001
- link right_palm:11: geometry collision mesh filename=package://nicoros/../../../urdf/meshes/right_palm_iam_583b2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 scale=0.001 0.001 0.001; visual mesh filename=package://nicoros/../../../urdf/meshes/right_palm_iam_583b2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 scale=0.001 0.001 0.001
- link right_shank:11: geometry collision mesh filename=package://nicoros/../../../urdf/meshes/right_shank_iam_7a73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 scale=0.001 0.001 0.001; visual mesh filename=package://nicoros/../../../urdf/meshes/right_shank_iam_7a73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 scale=0.001 0.001 0.001
- link right_shoulder:11: geometry collision mesh filename=package://nicoros/../../../urdf/meshes/right_shoulder_up_ia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 scale=0.001 0.001 0.001; visual mesh filename=package://nicoros/../../../urdf/meshes/right_shoulder_up_ia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 scale=0.001 0.001 0.001
- link right_thigh:11: geometry collision mesh filename=package://nicoros/../../../urdf/meshes/Thigh_right_complete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 scale=0.001 0.001 0.001; visual mesh filename=package://nicoros/../../../urdf/meshes/Thigh_right_complete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 scale=0.001 0.001 0.001
- link right_upper_arm:11: geometry collision mesh filename=package://nicoros/../../../urdf/meshes/right_lower_arm1_iam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 scale=0.001 0.001 0.001; visual mesh filename=package://nicoros/../../../urdf/meshes/right_lower_arm1_iam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 scale=0.001 0.001 0.001
- link torso:11: geometry collision mesh filename=package://nicoros/../../../urdf/meshes/torso_iam_fb80b350.S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 scale=0.001 0.001 0.001; visual mesh filename=package://nicoros/../../../urdf/meshes/torso_iam_fb80b350.S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 scale=0.001 0.001 0.001

File: api/src/nicomoveit/moveiturdf/urdf/complete_no_fingers.urdf (robot description, URDF)
Before this commit: robot complete, 28 links, 27 joints
Links:
- link head:21: geometry collision mesh filename=package://nicoros/../../../urdf/meshes/head_iam_b9cf2ea.STL scale=0.001 0.001 0.001; visual mesh filename=package://nicoros/../../../urdf/meshes/head_iam_b9cf2ea.STL scale=0.001 0.001 0.001
- link left_ankle:11: geometry collision mesh filename=package://nicoros/../../../urdf/meshes/right_ankle_MIR_iam_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 scale=0.001 0.001 0.001; visual mesh filename=package://nicoros/../../../urdf/meshes/right_ankle_MIR_iam_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 scale=0.001 0.001 0.001
- link left_foot:11: geometry collision mesh filename=package://nicoros/../../../urdf/meshes/left_foot_iam_620666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 scale=0.001 0.001 0.001; visual mesh filename=package://nicoros/../../../urdf/meshes/left_foot_iam_620666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 scale=0.001 0.001 0.001
- link left_hip_low:11: geometry collision mesh filename=package://nicoros/../../../urdf/meshes/right_hip_up2_MIR_ia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 scale=0.001 0.001 0.001; visual mesh filename=package://nicoros/../../../urdf/meshes/right_hip_up2_MIR_ia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 scale=0.001 0.001 0.001
- link left_hip_up:11: geometry collision mesh filename=package://nicoros/../../../urdf/meshes/right_hip_up_MIR_iam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 scale=0.001 0.001 0.001; visual mesh filename=package://nicoros/../../../urdf/meshes/right_hip_up_MIR_iam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 scale=0.001 0.001 0.001
- link left_lower_arm:11: geometry collision mesh filename=package://nicoros/../../../urdf/meshes/right_wrist_MIR_iam_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 scale=0.001 0.001 0.001; visual mesh filename=package://nicoros/../../../urdf/meshes/right_wrist_MIR_iam_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 scale=0.001 0.001 0.001
- link left_palm:11: geometry collision mesh filename=package://nicoros/../../../urdf/meshes/left_palm_iam_b92c61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 scale=0.001 0.001 0.001; visual mesh filename=package://nicoros/../../../urdf/meshes/left_palm_iam_b92c61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 scale=0.001 0.001 0.001
- link left_shank:11: geometry collision mesh filename=package://nicoros/../../../urdf/meshes/right_shank_MIR_iam_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 scale=0.001 0.001 0.001; visual mesh filename=package://nicoros/../../../urdf/meshes/right_shank_MIR_iam_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 scale=0.001 0.001 0.001
- link left_shoulder:11: geometry collision mesh filename=package://nicoros/../../../urdf/meshes/left_shoulder_up_iam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 scale=0.001 0.001 0.001; visual mesh filename=package://nicoros/../../../urdf/meshes/left_shoulder_up_iam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 scale=0.001 0.001 0.001
- link left_thigh:11: geometry collision mesh filename=package://nicoros/../../../urdf/meshes/Thigh_left_complete_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 scale=0.001 0.001 0.001; visual mesh filename=package://nicoros/../../../urdf/meshes/Thigh_left_complete_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 scale=0.001 0.001 0.001
- link left_upper_arm:11: geometry collision mesh filename=package://nicoros/../../../urdf/meshes/left_lower_arm_iam_5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 scale=0.001 0.001 0.001; visual mesh filename=package://nicoros/../../../urdf/meshes/left_lower_arm_iam_5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 scale=0.001 0.001 0.001
- link neck:11: geometry collision mesh filename=package://nicoros/../../../urdf/meshes/neck_iam_61141f4f.STL scale=0.001 0.001 0.001; visual mesh filename=package://nicoros/../../../urdf/meshes/neck_iam_61141f4f.STL scale=0.001 0.001 0.001
- link right_ankle:11: geometry collision mesh filename=package://nicoros/../../../urdf/meshes/right_ankle_iam_f4f7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 scale=0.001 0.001 0.001; visual mesh filename=package://nicoros/../../../urdf/meshes/right_ankle_iam_f4f7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 scale=0.001 0.001 0.001
- link right_foot:11: geometry collision mesh filename=package://nicoros/../../../urdf/meshes/right_foot_iam_3ff73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 scale=0.001 0.001 0.001; visual mesh filename=package://nicoros/../../../urdf/meshes/right_foot_iam_3ff73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 scale=0.001 0.001 0.001
- link right_hip_low:11: geometry collision mesh filename=package://nicoros/../../../urdf/meshes/right_hip_up2_iam_f4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 scale=0.001 0.001 0.001; visual mesh filename=package://nicoros/../../../urdf/meshes/right_hip_up2_iam_f4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 scale=0.001 0.001 0.001
- link right_hip_up:11: geometry collision mesh filename=package://nicoros/../../../urdf/meshes/right_hip_up_iam_f46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 scale=0.001 0.001 0.001; visual mesh filename=package://nicoros/../../../urdf/meshes/right_hip_up_iam_f46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 scale=0.001 0.001 0.001
- link right_lower_arm:11: geometry collision mesh filename=package://nicoros/../../../urdf/meshes/right_wrist_iam_771e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 scale=0.001 0.001 0.001; visual mesh filename=package://nicoros/../../../urdf/meshes/right_wrist_iam_771e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 scale=0.001 0.001 0.001
- link right_palm:11: geometry collision mesh filename=package://nicoros/../../../urdf/meshes/right_palm_iam_583b2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 scale=0.001 0.001 0.001; visual mesh filename=package://nicoros/../../../urdf/meshes/right_palm_iam_583b2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 scale=0.001 0.001 0.001
- link right_shank:11: geometry collision mesh filename=package://nicoros/../../../urdf/meshes/right_shank_iam_7a73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 scale=0.001 0.001 0.001; visual mesh filename=package://nicoros/../../../urdf/meshes/right_shank_iam_7a73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 scale=0.001 0.001 0.001
- link right_shoulder:11: geometry collision mesh filename=package://nicoros/../../../urdf/meshes/right_shoulder_up_ia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 scale=0.001 0.001 0.001; visual mesh filename=package://nicoros/../../../urdf/meshes/right_shoulder_up_ia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 scale=0.001 0.001 0.001
- link right_thigh:11: geometry collision mesh filename=package://nicoros/../../../urdf/meshes/Thigh_right_complete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 scale=0.001 0.001 0.001; visual mesh filename=package://nicoros/../../../urdf/meshes/Thigh_right_complete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 scale=0.001 0.001 0.001
- link right_upper_arm:11: geometry collision mesh filename=package://nicoros/../../../urdf/meshes/right_lower_arm1_iam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 scale=0.001 0.001 0.001; visual mesh filename=package://nicoros/../../../urdf/meshes/right_lower_arm1_iam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 scale=0.001 0.001 0.001
- link torso:11: geometry collision mesh filename=package://nicoros/../../../urdf/meshes/torso_iam_fb80b350.S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 scale=0.001 0.001 0.001; visual mesh filename=package://nicoros/../../../urdf/meshes/torso_iam_fb80b350.S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 scale=0.001 0.001 0.001
