Commit message: Updated inverse kinematics to use gaikpy, added visualizer and tests to nicomotion

File: api/src/nicomotion/scripts/nicomotion/urdf/kinematics.urdf (robot description, URDF)
Before this commit: robot complete, 45 links, 44 joints
Links:
- link finger_segment:11: geometry collision mesh filename=/home/connor/Dokumente/NICO-software/urdf/meshes/finger_seg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 scale=0.001 0.001 0.001; visual mesh filename=/home/connor/Dokumente/NICO-software/urdf/meshes/finger_seg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 scale=0.001 0.001 0.001
- link finger_segment:12: geometry collision mesh filename=/home/connor/Dokumente/NICO-software/urdf/meshes/finger_seg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 scale=0.001 0.001 0.001; visual mesh filename=/home/connor/Dokumente/NICO-software/urdf/meshes/finger_seg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 scale=0.001 0.001 0.001
- link finger_segment:13: geometry collision mesh filename=/home/connor/Dokumente/NICO-software/urdf/meshes/finger_seg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 scale=0.001 0.001 0.001; visual mesh filename=/home/connor/Dokumente/NICO-software/urdf/meshes/finger_seg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 scale=0.001 0.001 0.001
- link finger_segment:14: geometry collision mesh filename=/home/connor/Dokumente/NICO-software/urdf/meshes/finger_seg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 scale=0.001 0.001 0.001; visual mesh filename=/home/connor/Dokumente/NICO-software/urdf/meshes/finger_seg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 scale=0.001 0.001 0.001
- link finger_segment:15: geometry collision mesh filename=/home/connor/Dokumente/NICO-software/urdf/meshes/finger_seg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 scale=0.001 0.001 0.001; visual mesh filename=/home/connor/Dokumente/NICO-software/urdf/meshes/finger_seg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 scale=0.001 0.001 0.001
- link finger_segment:16: geometry collision mesh filename=/home/connor/Dokumente/NICO-software/urdf/meshes/finger_seg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 scale=0.001 0.001 0.001; visual mesh filename=/home/connor/Dokumente/NICO-software/urdf/meshes/finger_seg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 scale=0.001 0.001 0.001
- link finger_segment:21: geometry collision mesh filename=/home/connor/Dokumente/NICO-software/urdf/meshes/finger_seg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 scale=0.001 0.001 0.001; visual mesh filename=/home/connor/Dokumente/NICO-software/urdf/meshes/finger_seg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 scale=0.001 0.001 0.001
- link finger_segment:22: geometry collision mesh filename=/home/connor/Dokumente/NICO-software/urdf/meshes/finger_seg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 scale=0.001 0.001 0.001; visual mesh filename=/home/connor/Dokumente/NICO-software/urdf/meshes/finger_seg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 scale=0.001 0.001 0.001
- link finger_segment:23: geometry collision mesh filename=/home/connor/Dokumente/NICO-software/urdf/meshes/finger_seg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 scale=0.001 0.001 0.001; visual mesh filename=/home/connor/Dokumente/NICO-software/urdf/meshes/finger_seg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 scale=0.001 0.001 0.001
- link finger_segment:24: geometry collision mesh filename=/home/connor/Dokumente/NICO-software/urdf/meshes/finger_seg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 scale=0.001 0.001 0.001; visual mesh filename=/home/connor/Dokumente/NICO-software/urdf/meshes/finger_seg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 scale=0.001 0.001 0.001
- link finger_segment:25: geometry collision mesh filename=/home/connor/Dokumente/NICO-software/urdf/meshes/finger_seg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 scale=0.001 0.001 0.001; visual mesh filename=/home/connor/Dokumente/NICO-software/urdf/meshes/finger_seg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 scale=0.001 0.001 0.001
- link finger_segment:26: geometry collision mesh filename=/home/connor/Dokumente/NICO-software/urdf/meshes/finger_seg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 scale=0.001 0.001 0.001; visual mesh filename=/home/connor/Dokumente/NICO-software/urdf/meshes/finger_seg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 scale=0.001 0.001 0.001
- link fingertip:11: geometry collision mesh filename=/home/connor/Dokumente/NICO-software/urdf/meshes/fingertip_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 scale=0.001 0.001 0.001; visual mesh filename=/home/connor/Dokumente/NICO-software/urdf/meshes/fingertip_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 scale=0.001 0.001 0.001
- link fingertip:12: geometry collision mesh filename=/home/connor/Dokumente/NICO-software/urdf/meshes/fingertip_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 scale=0.001 0.001 0.001; visual mesh filename=/home/connor/Dokumente/NICO-software/urdf/meshes/fingertip_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 scale=0.001 0.001 0.001
- link fingertip:13: geometry collision mesh filename=/home/connor/Dokumente/NICO-software/urdf/meshes/fingertip_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 scale=0.001 0.001 0.001; visual mesh filename=/home/connor/Dokumente/NICO-software/urdf/meshes/fingertip_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 scale=0.001 0.001 0.001
- link fingertip:14: geometry collision mesh filename=/home/connor/Dokumente/NICO-software/urdf/meshes/fingertip_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 scale=0.001 0.001 0.001; visual mesh filename=/home/connor/Dokumente/NICO-software/urdf/meshes/fingertip_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 scale=0.001 0.001 0.001
- link fingertip:15: geometry collision mesh filename=/home/connor/Dokumente/NICO-software/urdf/meshes/fingertip_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 scale=0.001 0.001 0.001; visual mesh filename=/home/connor/Dokumente/NICO-software/urdf/meshes/fingertip_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 scale=0.001 0.001 0.001
- link fingertip:16: geometry collision mesh filename=/home/connor/Dokumente/NICO-software/urdf/meshes/fingertip_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 scale=0.001 0.001 0.001; visual mesh filename=/home/connor/Dokumente/NICO-software/urdf/meshes/fingertip_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 scale=0.001 0.001 0.001
- link head:21: geometry collision mesh filename=/home/connor/Dokumente/NICO-software/urdf/meshes/head_iam_b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 scale=0.001 0.001 0.001; visual mesh filename=/home/connor/Dokumente/NICO-software/urdf/meshes/head_iam_b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 scale=0.001 0.001 0.001
- link left_ankle:11: geometry collision mesh filename=/home/connor/Dokumente/NICO-software/urdf/meshes/right_ankl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 scale=0.001 0.001 0.001; visual mesh filename=/home/connor/Dokumente/NICO-software/urdf/meshes/right_ankl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 scale=0.001 0.001 0.001
- link left_collarbone:11: geometry collision mesh filename=/home/connor/Dokumente/NICO-software/urdf/meshes/left_upper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 scale=0.001 0.001 0.001; visual mesh filename=/home/connor/Dokumente/NICO-software/urdf/meshes/left_upper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 scale=0.001 0.001 0.001
- link left_foot:11: geometry collision mesh filename=/home/connor/Dokumente/NICO-software/urdf/meshes/left_foot_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 scale=0.001 0.001 0.001; visual mesh filename=/home/connor/Dokumente/NICO-software/urdf/meshes/left_foot_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 scale=0.001 0.001 0.001
- link left_hip_low:11: geometry collision mesh filename=/home/connor/Dokumente/NICO-software/urdf/meshes/right_hip_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 scale=0.001 0.001 0.001; visual mesh filename=/home/connor/Dokumente/NICO-software/urdf/meshes/right_hip_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 scale=0.001 0.001 0.001
- link left_hip_up:11: geometry collision mesh filename=/home/connor/Dokumente/NICO-software/urdf/meshes/right_hip_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 scale=0.001 0.001 0.001; visual mesh filename=/home/connor/Dokumente/NICO-software/urdf/meshes/right_hip_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 scale=0.001 0.001 0.001
- link left_lower_arm:11: geometry collision mesh filename=/home/connor/Dokumente/NICO-software/urdf/meshes/right_wris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 scale=0.001 0.001 0.001; visual mesh filename=/home/connor/Dokumente/NICO-software/urdf/meshes/right_wris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 scale=0.001 0.001 0.001
- link left_palm:11: geometry collision mesh filename=/home/connor/Dokumente/NICO-software/urdf/meshes/left_palm_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 scale=0.001 0.001 0.001; visual mesh filename=/home/connor/Dokumente/NICO-software/urdf/meshes/left_palm_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 scale=0.001 0.001 0.001
- link left_shank:11: geometry collision mesh filename=/home/connor/Dokumente/NICO-software/urdf/meshes/right_shan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 scale=0.001 0.001 0.001; visual mesh filename=/home/connor/Dokumente/NICO-software/urdf/meshes/right_shan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 scale=0.001 0.001 0.001
- link left_shoulder:11: geometry collision mesh filename=/home/connor/Dokumente/NICO-software/urdf/meshes/left_shoul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 scale=0.001 0.001 0.001; visual mesh filename=/home/connor/Dokumente/NICO-software/urdf/meshes/left_shoul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 scale=0.001 0.001 0.001
- link left_thigh:11: geometry collision mesh filename=/home/connor/Dokumente/NICO-software/urdf/meshes/Thigh_left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 scale=0.001 0.001 0.001; visual mesh filename=/home/connor/Dokumente/NICO-software/urdf/meshes/Thigh_left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 scale=0.001 0.001 0.001
- link left_upper_arm:11: geometry collision mesh filename=/home/connor/Dokumente/NICO-software/urdf/meshes/left_lower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 scale=0.001 0.001 0.001; visual mesh filename=/home/connor/Dokumente/NICO-software/urdf/meshes/left_lower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 scale=0.001 0.001 0.001
- link left_wrist:11: geometry collision mesh filename=/home/connor/Dokumente/NICO-software/urdf/meshes/left_wrist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 scale=0.001 0.001 0.001; visual mesh filename=/home/connor/Dokumente/NICO-software/urdf/meshes/left_wrist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 scale=0.001 0.001 0.001
- link neck:11: geometry collision mesh filename=/home/connor/Dokumente/NICO-software/urdf/meshes/neck_iam_6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 scale=0.001 0.001 0.001; visual mesh filename=/home/connor/Dokumente/NICO-software/urdf/meshes/neck_iam_6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 scale=0.001 0.001 0.001
- link right_ankle:11: geometry collision mesh filename=/home/connor/Dokumente/NICO-software/urdf/meshes/right_ankl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 scale=0.001 0.001 0.001; visual mesh filename=/home/connor/Dokumente/NICO-software/urdf/meshes/right_ankl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 scale=0.001 0.001 0.001
- link right_collarbone:11: geometry collision mesh filename=/home/connor/Dokumente/NICO-software/urdf/meshes/right_uppe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 scale=0.001 0.001 0.001; visual mesh filename=/home/connor/Dokumente/NICO-software/urdf/meshes/right_uppe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 scale=0.001 0.001 0.001
- link right_foot:11: geometry collision mesh filename=/home/connor/Dokumente/NICO-software/urdf/meshes/right_foot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 scale=0.001 0.001 0.001; visual mesh filename=/home/connor/Dokumente/NICO-software/urdf/meshes/right_foot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 scale=0.001 0.001 0.001
- link right_hip_low:11: geometry collision mesh filename=/home/connor/Dokumente/NICO-software/urdf/meshes/right_hip_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 scale=0.001 0.001 0.001; visual mesh filename=/home/connor/Dokumente/NICO-software/urdf/meshes/right_hip_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 scale=0.001 0.001 0.001
- link right_hip_up:11: geometry collision mesh filename=/home/connor/Dokumente/NICO-software/urdf/meshes/right_hip_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 scale=0.001 0.001 0.001; visual mesh filename=/home/connor/Dokumente/NICO-software/urdf/meshes/right_hip_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 scale=0.001 0.001 0.001
- link right_lower_arm:11: geometry collision mesh filename=/home/connor/Dokumente/NICO-software/urdf/meshes/right_wris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 scale=0.001 0.001 0.001; visual mesh filename=/home/connor/Dokumente/NICO-software/urdf/meshes/right_wris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 scale=0.001 0.001 0.001
- link right_palm:11: geometry collision mesh filename=/home/connor/Dokumente/NICO-software/urdf/meshes/right_palm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 scale=0.001 0.001 0.001; visual mesh filename=/home/connor/Dokumente/NICO-software/urdf/meshes/right_palm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 scale=0.001 0.001 0.001
- link right_shank:11: geometry collision mesh filename=/home/connor/Dokumente/NICO-software/urdf/meshes/right_shan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 scale=0.001 0.001 0.001; visual mesh filename=/home/connor/Dokumente/NICO-software/urdf/meshes/right_shan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 scale=0.001 0.001 0.001
- link right_shoulder:11: geometry collision mesh filename=/home/connor/Dokumente/NICO-software/urdf/meshes/right_shou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 scale=0.001 0.001 0.001; visual mesh filename=/home/connor/Dokumente/NICO-software/urdf/meshes/right_shou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 scale=0.001 0.001 0.001
- link right_thigh:11: geometry collision mesh filename=/home/connor/Dokumente/NICO-software/urdf/meshes/Thigh_righ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 scale=0.001 0.001 0.001; visual mesh filename=/home/connor/Dokumente/NICO-software/urdf/meshes/Thigh_righ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 scale=0.001 0.001 0.001
- link right_upper_arm:11: geometry collision mesh filename=/home/connor/Dokumente/NICO-software/urdf/meshes/right_lowe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 scale=0.001 0.001 0.001; visual mesh filename=/home/connor/Dokumente/NICO-software/urdf/meshes/right_lowe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 scale=0.001 0.001 0.001
- link right_wrist:11: geometry collision mesh filename=/home/connor/Dokumente/NICO-software/urdf/meshes/right_wris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 scale=0.001 0.001 0.001; visual mesh filename=/home/connor/Dokumente/NICO-software/urdf/meshes/right_wris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 scale=0.001 0.001 0.001
- link torso:11: geometry collision mesh filename=/home/connor/Dokumente/NICO-software/urdf/meshes/torso_iam_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 scale=0.001 0.001 0.001; visual mesh filename=/home/connor/Dokumente/NICO-software/urdf/meshes/torso_iam_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 scale=0.001 0.001 0.001
